File: PCB/Mailbox Notifier 2.2.brd (EAGLE design)
At the start: 50 x 50 mm, 12 parts, among them Q1 MOSFET-NCHANNEL2N7000

Commit message: Final Eagle files
Parts:
- added R4: 1K, SparkFun-Passives:AXIAL-0.4
Connections:
- new net N$7: H3.1, R4.P$1
- net 5V: now also R4.P$2; no longer H3.1
Routing:
- net 5V: track 58.3 -> 40.3 mm
- net N$7: track 0.00 -> 13.4 mm
Other:
- board text added: "Rom3oDelta7"
Changed lines of the file:
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@@
 CC-BY-SA 4.0
 </text>
+<text x="26.035" y="-11.43" size="1.778" layer="51">Rom3oDelta7</text>
 </plain>
 <attributes>
@@
 <attribute name="NAME" x="11.811" y="32.512" size="1.27" layer="25" ratio="10" rot="R270"/>
 </element>
+<element name="R4" library="SparkFun-Passives" package="AXIAL-0.4" value="1K" x="42.2275" y="12.7" rot="R270"/>
 </elements>
 <signals>
@@
 <contactref element="U$1" pad="5V"/>
 <contactref element="H2" pad="2"/>
-<contactref element="H3" pad="1"/>
+<contactref element="R4" pad="P$2"/>
 <wire x1="33.1089" y1="5.1689" x2="5.1689" y2="5.1689" width="0.6096" layer="1"/>
-<wire x1="37.9984" y1="10.0584" x2="33.1089" y2="5.1689" width="0.6096" layer="1"/>
+<wire x1="38.1" y1="10.16" x2="33.1089" y2="5.1689" width="0.6096" layer="1"/>
 <wire x1="5.1689" y1="5.1689" x2="5.08" y2="5.08" width="0.6096" layer="1"/>
-<wire x1="37.9984" y1="10.0584" x2="38.1" y2="10.16" width="0.6096" layer="1"/>
-<wire x1="43.7261" y1="15.0876" x2="43.7261" y2="30.4546" width="0.6096" layer="1"/>
-<wire x1="38.9763" y1="10.3378" x2="43.7261" y2="15.0876" width="0.6096" layer="1"/>
-<wire x1="38.2778" y1="10.3378" x2="38.9763" y2="10.3378" width="0.6096" layer="1"/>
-<wire x1="43.7261" y1="30.4546" x2="43.815" y2="30.48" width="0.6096" layer="1"/>
-<wire x1="38.2778" y1="10.3378" x2="38.1" y2="10.16" width="0.6096" layer="1"/>
+<wire x1="40.513" y1="7.6835" x2="42.1894" y2="7.6835" width="0.6096" layer="1"/>
+<wire x1="38.2778" y1="9.9187" x2="40.513" y2="7.6835" width="0.6096" layer="1"/>
+<wire x1="42.1894" y1="7.6835" x2="42.2275" y2="7.62" width="0.6096" layer="1"/>
+<wire x1="38.2778" y1="9.9187" x2="38.1" y2="10.16" width="0.6096" layer="1"/>
 </signal>
 <signal name="GND" class="1">
@@
 <wire x1="11.7348" y1="23.749" x2="13.97" y2="21.5138" width="0.3048" layer="1"/>
 <wire x1="11.7348" y1="30.1752" x2="11.7348" y2="23.749" width="0.3048" layer="1"/>
-<wire x1="5.1689" y1="36.7411" x2="11.7348" y2="30.1752" width="0.3048" layer="1"/>
+<wire x1="5.08" y1="36.83" x2="11.7348" y2="30.1752" width="0.3048" layer="1"/>
 <wire x1="15.2273" y1="20.3962" x2="15.24" y2="20.32" width="0.3048" layer="1"/>
-<wire x1="5.1689" y1="36.7411" x2="5.08" y2="36.83" width="0.3048" layer="1"/>
 </signal>
 <signal name="N$4">
@@
 <wire x1="46.3804" y1="30.4546" x2="46.355" y2="30.48" width="0.3048" layer="1"/>
 <wire x1="46.3804" y1="17.8816" x2="46.355" y2="17.78" width="0.3048" layer="1"/>
-<wire x1="44.5643" y1="32.6898" x2="44.5643" y2="43.7261" width="0.3048" layer="1"/>
-<wire x1="46.2407" y1="31.0134" x2="44.5643" y2="32.6898" width="0.3048" layer="1"/>
-<wire x1="46.2407" y1="30.5943" x2="46.2407" y2="31.0134" width="0.3048" layer="1"/>
+<wire x1="44.5643" y1="32.2707" x2="44.5643" y2="43.7261" width="0.3048" layer="1"/>
+<wire x1="46.355" y1="30.48" x2="44.5643" y2="32.2707" width="0.3048" layer="1"/>
 <wire x1="44.5643" y1="43.7261" x2="44.45" y2="43.815" width="0.3048" layer="1"/>
-<wire x1="46.2407" y1="30.5943" x2="46.355" y2="30.48" width="0.3048" layer="1"/>
 </signal>
 <signal name="N$5" class="1">
@@
 <wire x1="42.1894" y1="42.1894" x2="42.1894" y2="41.7703" width="0.6096" layer="1"/>
 <wire x1="42.1894" y1="41.7703" x2="42.1894" y2="23.749" width="0.6096" layer="1"/>
-<wire x1="42.4688" y1="42.4688" x2="42.1894" y2="42.1894" width="0.6096" layer="1"/>
+<wire x1="42.545" y1="42.545" x2="42.1894" y2="42.1894" width="0.6096" layer="1"/>
 <wire x1="38.1381" y1="20.3962" x2="38.1" y2="20.32" width="0.6096" layer="1"/>
-<wire x1="42.4688" y1="42.4688" x2="42.545" y2="42.545" width="0.6096" layer="1"/>
 <wire x1="21.7932" y1="43.1673" x2="18.4404" y2="43.1673" width="0.6096" layer="1"/>
 <wire x1="23.1902" y1="41.7703" x2="21.7932" y2="43.1673" width="0.6096" layer="1"/>
-<wire x1="41.91" y1="41.7703" x2="23.1902" y2="41.7703" width="0.6096" layer="1"/>
+<wire x1="42.1894" y1="41.7703" x2="23.1902" y2="41.7703" width="0.6096" layer="1"/>
 <wire x1="18.4404" y1="43.1673" x2="18.415" y2="43.18" width="0.6096" layer="1"/>
-<wire x1="41.91" y1="41.7703" x2="42.1894" y2="41.7703" width="0.6096" layer="1"/>
 </signal>
 <signal name="N$1" class="1">
@@
 <wire x1="8.382" y1="43.1673" x2="8.255" y2="43.18" width="0.6096" layer="1"/>
 </signal>
+<signal name="N$7">
+<contactref element="R4" pad="P$1"/>
+<contactref element="H3" pad="1"/>
+<wire x1="43.7261" y1="19.2786" x2="43.7261" y2="30.4546" width="0.3048" layer="1"/>
+<wire x1="42.2275" y1="17.78" x2="43.7261" y2="19.2786" width="0.3048" layer="1"/>
+<wire x1="43.7261" y1="30.4546" x2="43.815" y2="30.48" width="0.3048" layer="1"/>
+</signal>
 </signals>
